Commit message: .

File: Myhal_Simulator/nav_noetic_ws/src/jackal_velodyne/urdf/jackal_velodyne.urdf.xacro (robot description, xacro)
@@ -313,8 +313,3 @@
     </VLP-16>
   </xacro:unless>
-  <xacro:include filename="$(find kinect_v2)/urdf/kinect_v2.urdf.xacro" />
-    <xacro:kinect_v2  parent="support_link3">
-        <origin xyz="0 0 -0.04"
-                rpy="0 0 0" />
-   </xacro:kinect_v2>
 </robot>
